File: pcbs/controller_overlay.kicad_pcb (KiCad board)
At the start: 2 copper layers, 19.7 x 60.1 mm, 2 parts

Commit message: ordered and working nicely.. need some adjustments
Parts:
- moved MH1 23.9 mm to (185.0, 107.7)
- moved MH2 22.5 mm to (201.0, 116.6)
Other:
- board size 19.7 x 60.1 mm -> 22 x 62.8 mm
